Commit message: update panda to be consistent with my def, update gp4 joint limit and collision

File: resources/gp4/gp4_spherized.urdf (robot description, URDF)
Before this commit: robot Yaskawa_gp4, 12 links, 11 joints
Joints:
- joint joint_3: limit lower=-1.1344640137963142 upper=3.490658503988659 effort=200 velocity=2 -> lower=-0.99 upper=3.30 effort=200 velocity=2

File: resources/panda/panda_spherized.urdf (robot description, URDF)
Before this commit: robot panda, 13 links, 12 joints
Joints:
- joint panda_finger_joint1: origin xyz=0 0.065 0.0584 rpy=0 0 0 -> xyz=0 0.0 0.0584 rpy=0 0 0
- joint panda_finger_joint2: origin xyz=0 -0.065 0.0584 rpy=0 0 0 -> xyz=0 0.0 0.0584 rpy=0 0 0
- joint panda_hand_joint: origin xyz=0 0 0 rpy=0 0 -0.785398163397 -> xyz=0 0 0 rpy=0 0 0

Commit message: update gp4 spheres

File: resources/gp4/gp4_spherized.urdf (robot description, URDF)
Before this commit: robot Yaskawa_gp4, 12 links, 11 joints
Links:
- link base_link: geometry collision sphere radius=0.067458; collision sphere radius=0.08014
- link fts: geometry collision sphere radius=0.035668; collision sphere radius=0.036558
- link link_1: geometry collision sphere radius=0.090185; collision sphere radius=0.096502
- link link_3: geometry collision sphere radius=0.052807; collision sphere radius=0.072948
- link link_5: geometry collision sphere radius=0.044263; collision sphere radius=0.048512
- link link_6: geometry collision sphere radius=0.022052; collision sphere radius=0.022972
- link link_tool: geometry collision sphere radius=0.003; collision sphere radius=0.003
